File: 2026_12_2Wheel_Balance_Robot_v1_LAYOUT/2026_12_2Wheel_Balance_Robot_v1/2026_12_2Wheel_Balance_Robot_v1.kicad_pcb (KiCad board)
At the start: 2 copper layers, 68.6 x 53.4 mm, 56 parts, among them J1 Conn_01x04, J2 CONN_MPU6050, J3 USB_C_Receptacle_USB2.0_14P, J4 ESP_Conn, J5 BATT_CONN, J6 M1_CONN, J7 M2_CONN, J8 ENCODER_CONN, J9 MT6701_CONN, SW2 SW_uP_Reset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

Commit message: update gerber
Routing:
- net GND: track 61.5 -> 64.2 mm
- net +5V: track 83.7 -> 83.0 mm
Changed lines of the file:
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@@
 		(tags "capacitor handsolder")
 		(property "Reference" "C26"
-			(at -3.4798 -0.127 0)
+			(at -1.7022 -2.0346 0)
 			(layer "F.SilkS")
 			(effects
@@
 	)
 	(gr_text "IMU (MPU6050)"
-		(at 138.6209 105.2668 0)
+		(at 137.4459 105.5168 0)
 		(layer "F.SilkS")
 		(effects
@@
 	)
 	(segment
+		(start 103.6209 102.4168)
+		(end 103.6209 101.5444)
+		(width 0.508)
+		(layer "F.Cu")
+		(net "GND")
+	)
+	(segment
 		(start 138.8555 66.5822)
 		(end 138.8709 66.5668)
@@
 	)
 	(segment
+		(start 161.6765 83.6508)
+		(end 161.7585 83.7328)
+		(width 0.508)
+		(layer "F.Cu")
+		(net "GND")
+	)
+	(segment
 		(start 122.3385 91.0844)
 		(end 122.3209 91.0668)
@@
 	)
 	(segment
+		(start 162.7209 87.0668)
+		(end 161.1053 87.0668)
+		(width 0.508)
+		(layer "F.Cu")
+		(net "GND")
+	)
+	(segment
 		(start 151.4209 92.4668)
 		(end 150.3216 92.4668)
@@
 	)
 	(segment
+		(start 161.1053 87.0668)
+		(end 161.0928 87.0793)
+		(width 0.508)
+		(layer "F.Cu")
+		(net "GND")
+	)
+	(segment
 		(start 121.7144 78.9178)
 		(end 120.3851 78.9178)
@@
 	)
 	(segment
-		(start 161.0928 88.6449)
-		(end 161.0709 88.6668)
-		(width 0.381)
-		(layer "F.Cu")
-		(net "GND")
-	)
-	(segment
 		(start 160.5306 76.3571)
 		(end 160.3209 76.5668)
@@
 	)
 	(segment
-		(start 104.6707 101.3206)
-		(end 104.7809 101.4308)
-		(width 0.381)
-		(layer "F.Cu")
-		(net "GND")
-	)
-	(segment
 		(start 109.2537 102.4128)
 		(end 109.2537 101.022)
@@
 	)
 	(segment
-		(start 150.9449 85.307)
-		(end 150.9449 86.4428)
-		(width 0.381)
+		(start 157.453 83.6508)
+		(end 157.5206 83.7184)
+		(width 0.508)
 		(layer "F.Cu")
 		(net "GND")
 	)
 	(segment
-		(start 161.0928 87.0793)
-		(end 161.0928 88.6449)
+		(start 150.9449 85.307)
+		(end 150.9449 86.4428)
 		(width 0.381)
 		(layer "F.Cu")
@@
 	)
 	(segment
+		(start 160.9149 83.6508)
+		(end 161.6765 83.6508)
+		(width 0.508)
+		(layer "F.Cu")
+		(net "GND")
+	)
+	(segment
 		(start 111.048 89.9922)
 		(end 109.8695 89.9922)
@@
 	)
 	(segment
+		(start 137.9709 108.0918)
+		(end 137.7781 108.0918)
+		(width 0.508)
+		(layer "F.Cu")
+		(net "GND")
+	)
+	(segment
 		(start 108.5053 86.7844)
 		(end 108.5909 86.6988)
@@
 	)
 	(segment
-		(start 103.3971 101.3206)
-		(end 104.6707 101.3206)
-		(width 0.381)
-		(layer "F.Cu")
-		(net "GND")
-	)
-	(segment
 		(start 138.9063 73.0458)
 		(end 138.9185 73.0336)
@@
 		(net "GND")
 	)
+	(segment
+		(start 156.7209 83.6508)
+		(end 157.453 83.6508)
+		(width 0.508)
+		(layer "F.Cu")
+		(net "GND")
+	)
+	(segment
+		(start 137.7781 108.0918)
+		(end 137.0521 107.3658)
+		(width 0.508)
+		(layer "F.Cu")
+		(net "GND")
+	)
+	(segment
+		(start 103.6209 101.5444)
+		(end 103.3971 101.3206)
+		(width 0.508)
+		(layer "F.Cu")
+		(net "GND")
+	)
 	(via
 		(at 141.1029 66.5168)
@@
 	)
 	(via
-		(at 137.0389 106.0028)
+		(at 137.9709 108.0918)
 		(size 0.6)
 		(drill 0.3)
@@
 	)
 	(via
-		(at 104.7809 101.4308)
+		(at 103.6209 102.4168)
 		(size 0.6)
 		(drill 0.3)
@@
 	)
 	(via
-		(at 156.8509 83.6508)
+		(at 156.7209 83.6508)
 		(size 0.6)
 		(drill 0.3)
@@
 	)
 	(via
-		(at 161.0709 88.6668)
+		(at 162.7209 87.0668)
 		(size 0.6)
 		(drill 0.3)
@@
 	)
 	(segment
-		(start 151.3709 73.8644)
-		(end 150.9153 73.8644)
-		(width 0.381)
-		(layer "F.Cu")
-		(net "+5V")
-	)
-	(segment
 		(start 149.6209 88.231)
 		(end 147.6449 90.207)
@@
 	)
 	(segment
-		(start 150.9153 73.8644)
-		(end 149.6209 75.1588)
+		(start 150.9209 70.752209)
+		(end 150.9209 73.8644)
 		(width 0.381)
 		(layer "F.Cu")
@@
 	)
 	(segment
+		(start 150.9209 73.8644)
+		(end 150.9153 73.8644)
+		(width 0.381)
+		(layer "F.Cu")
+		(net "+5V")
+	)
+	(segment
 		(start 152.9709 109.2168)
 		(end 135.4709 109.2168)
@@
 	)
 	(segment
-		(start 151.3709 71.202209)
-		(end 151.3709 73.8644)
-		(width 0.381)
-		(layer "F.Cu")
-		(net "+5V")
-	)
-	(segment
-		(start 150.3789 70.210209)
-		(end 151.3709 71.202209)
+		(start 150.9153 73.8644)
+		(end 149.6209 75.1588)
 		(width 0.381)
 		(layer "F.Cu")
@@
 	)
 	(segment
+		(start 150.3789 70.210209)
+		(end 150.9209 70.752209)
+		(width 0.381)
+		(layer "F.Cu")
+		(net "+5V")
+	)
+	(segment
 		(start 147.6449 90.207)
 		(end 147.8807 90.207)
@@
 		(start 137.0209 100.4668)
 		(end 137.0209 92.163408)
-		(width 0.254)
+		(width 0.3048)
 		(layer "F.Cu")
 		(net "/IMU_INT")
@@
 		(start 141.7709 105.2168)
 		(end 137.0209 100.4668)
-		(width 0.254)
+		(width 0.3048)
 		(layer "F.Cu")
 		(net "/IMU_INT")
@@
 		(start 152.2921 107.3658)
 		(end 150.1431 105.2168)
-		(width 0.254)
+		(width 0.3048)
 		(layer "F.Cu")
 		(net "/IMU_INT")
@@
 		(start 150.1431 105.2168)
 		(end 141.7709 105.2168)
-		(width 0.254)
+		(width 0.3048)
 		(layer "F.Cu")
 		(net "/IMU_INT")
