File: 2026_12_2Wheel_Balance_Robot_v1_LAYOUT/2026_12_2Wheel_Balance_Robot_v1/2026_12_2Wheel_Balance_Robot_v1.kicad_pcb (KiCad board)
At the start: 2 copper layers, 68.6 x 53.4 mm, 56 parts, among them J1 Conn_01x04, J2 CONN_MPU6050, J3 USB_C_Receptacle_USB2.0_14P, J4 ESP_Conn, J5 BATT_CONN, J6 M1_CONN, J7 M2_CONN, J8 ENCODER_CONN, J9 MT6701_CONN, SW2 SW_uP_Reset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

Commit message: update gerber
Other:
- board text added: "2 Wheel Robot Charlie Shields ENCE-3231 Spring 2026"
- board text removed: "Charlie Shields ENCE-3231 Spring 2026"
Changed lines of the file:
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@@
 		)
 	)
-	(gr_text "Charlie Shields\nENCE-3231 Spring 2026"
-		(at 165.8209 66.3668 0)
+	(gr_text "2 Wheel Robot\nCharlie Shields\nENCE-3231 Spring 2026"
+		(at 165.9709 66.6168 0)
 		(layer "B.SilkS")
 		(effects

Commit message: add drill files
Routing:
- net /ENC_A: track 21.3 -> 23.3 mm
- net /ENC_B: track 23.3 -> 25.2 mm
Changed lines of the file:
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@@
 	)
 	(gr_text "ESP CONN"
-		(at 103.2709 76.5668 90)
+		(at 111.6459 77.8668 90)
 		(layer "F.SilkS")
 		(effects
@@
 	)
 	(segment
-		(start 130.1713 93.5094)
-		(end 130.1713 94.354992)
+		(start 130.1713 97.6664)
+		(end 128.3709 99.4668)
 		(width 0.254)
 		(layer "F.Cu")
@@
 	)
 	(segment
-		(start 130.1713 94.354992)
-		(end 125.059492 99.4668)
+		(start 111.7537 101.234)
+		(end 111.7537 102.4128)
 		(width 0.254)
 		(layer "F.Cu")
@@
 	)
 	(segment
-		(start 125.059492 99.4668)
-		(end 114.6997 99.4668)
+		(start 113.5169 99.4708)
+		(end 111.7537 101.234)
 		(width 0.254)
 		(layer "F.Cu")
@@
 	)
 	(segment
-		(start 111.7537 101.234)
-		(end 111.7537 102.4128)
+		(start 128.3709 99.4668)
+		(end 114.6997 99.4668)
 		(width 0.254)
 		(layer "F.Cu")
@@
 	)
 	(segment
-		(start 113.5169 99.4708)
-		(end 111.7537 101.234)
+		(start 114.695699 99.4708)
+		(end 113.5169 99.4708)
 		(width 0.254)
 		(layer "F.Cu")
@@
 	)
 	(segment
-		(start 114.695699 99.4708)
-		(end 113.5169 99.4708)
+		(start 130.1713 93.5094)
+		(end 130.1713 97.6664)
 		(width 0.254)
 		(layer "F.Cu")
@@
 	)
 	(segment
-		(start 130.6483 94.377992)
-		(end 130.6253 94.400992)
+		(start 130.6713 93.5094)
+		(end 130.6483 93.5094)
 		(width 0.254)
 		(layer "F.Cu")
@@
 	)
 	(segment
-		(start 125.201545 99.9668)
-		(end 115.6709 99.9668)
+		(start 130.6253 97.9624)
+		(end 128.6209 99.9668)
 		(width 0.254)
 		(layer "F.Cu")
@@
 	)
 	(segment
-		(start 114.2537 101.384)
-		(end 114.2537 102.4128)
+		(start 115.6709 99.9668)
+		(end 114.2537 101.384)
 		(width 0.254)
 		(layer "F.Cu")
@@
 	)
 	(segment
-		(start 130.6253 94.543045)
-		(end 125.201545 99.9668)
+		(start 130.6253 94.400992)
+		(end 130.6253 97.9624)
 		(width 0.254)
 		(layer "F.Cu")
@@
 	)
 	(segment
-		(start 115.6709 99.9668)
-		(end 114.2537 101.384)
+		(start 128.6209 99.9668)
+		(end 115.6709 99.9668)
 		(width 0.254)
 		(layer "F.Cu")
@@
 	)
 	(segment
-		(start 130.6253 94.400992)
-		(end 130.6253 94.543045)
+		(start 114.2537 101.384)
+		(end 114.2537 102.4128)
 		(width 0.254)
 		(layer "F.Cu")
@@
 	)
 	(segment
-		(start 130.6713 93.5094)
-		(end 130.6483 93.5094)
+		(start 130.6483 94.377992)
+		(end 130.6253 94.400992)
 		(width 0.254)
 		(layer "F.Cu")
